Commit message: Joysick mapping, ROS service added to launch file, URDF warning fixed

File: legged_examples/legged_unitree/legged_unitree_description/urdf/robot.xacro (robot description, xacro)
@@ -7,7 +7,12 @@
     <xacro:include filename="$(find legged_unitree_description)/urdf/common/imu.xacro"/>
     <xacro:include filename="$(find legged_unitree_description)/urdf/$(arg robot_type)/const.xacro"/>
-<!--    <xacro:property name="mesh_path" value="../meshes"/>-->
-    <xacro:property name="mesh_path" value="$(find legged_unitree_description)/meshes/$(arg robot_type)"/>
-    <link name="base">
+   <!--    <xacro:property name="mesh_path" value="../meshes"/>-->
+   <xacro:property name="mesh_path" value="package://$(arg robot_type)_description/meshes"/>
+    <link name="base"/>
+    <joint name="base_inertia_joint" type="fixed">
+      <parent link="base"/>
+      <child link="base_inertia" />
+    </joint>
+    <link name="base_inertia">
         <visual>
             <origin rpy="0 0 0" xyz="0 0 0"/>
